File: 2 - CPU and memory card with the essentials (rev 2)/2 - CPU and memory card with the essentials (rev 2).kicad_pcb (KiCad board)
At the start: 2 copper layers, 152.3 x 106.7 mm, 55 parts, among them J1 BUS 1, J10 RX BUS DIS, J11 TX BUS DIS, J12 LPT or Keyboard, J2 MODE 2, J3 SIO CLK, J4 COM1: DCE, J5 RTS/CTR DIR, J6 VCC DIS, J7 COM2: TTL, J8 DATA DIR, J9 DTR|RTS/CTS, U1 74HC74, U10 AS6C4008, U11 AS6C4008, U12 Z84C3010 CTC, U13 MAX232, U14 Z84C4010, U15 Z84C20xx PIO, U2 ATF22V10C, U3 ATF22V10C, U4 ATF22V10C, U5 ATF22V10C, U6 74HCT573, U7 74HCT573, U8 Z84C0010, U9 SST39SF010, X1 20 MHz, X2 3.6864 MHz

Commit message: Updated disk activity circuit in mother board, and improved layout in CPU card
Parts:
- removed J10: RX BUS DIS, Connector_PinHeader_2.54mm:PinHeader_1x02_P2.54mm_Vertical
- removed J12: LPT or Keyboard, Connector_Dsub:DSUB-25_Female_Horizontal_P2.77x2.84mm_EdgePinOffset4.94mm_Housed_MountingHolesOffset7.48mm
- removed R1, R2, R3: 3K3, Resistor_THT:R_Axial_DIN0207_L6.3mm_D2.5mm_P10.16mm_Horizontal
- added AFF1: HI BANK #, Display_7Segment:7SegmentLED_LTS6760_LTS6780, F.Cu at (83.2, 43.8)
- added AFF2: LO BANK #, Display_7Segment:7SegmentLED_LTS6760_LTS6780, F.Cu at (95.9, 43.8)
- added BAR1: STATUS, 0_Library:BAR_GRAPH_8, F.Cu at (85.7, 111.1)
- added C21: 0.1µF, Capacitor_THT:C_Disc_D3.0mm_W1.6mm_P2.50mm, F.Cu at (82.5, 63.5)
- added C22: 0.1µF, Capacitor_THT:C_Disc_D3.0mm_W1.6mm_P2.50mm, F.Cu at (137.2, 34.9)
- added D1: 1N5819, Diode_THT:D_DO-41_SOD81_P10.16mm_Horizontal, F.Cu at (139.1, 74.3)
- added RN7: 3K3, Resistor_THT:R_Array_SIP7, F.Cu at (214.0, 90.8)
- added U16: 74HCT563, Package_DIP:DIP-20_W7.62mm_Socket, F.Cu at (85.7, 95.9)
- C13, C14, C15: value 1uF -> 0.1µF
- C17, C18, C19: value 0.1µF -> 1uF
- C9: value 0.1uF -> 0.1µF; footprint Capacitor_THT:C_Disc_D3.0mm_W2.0mm_P2.50mm -> Capacitor_THT:C_Disc_D3.0mm_W1.6mm_P2.50mm
- J11: value TX BUS DIS -> COM1: DCE; footprint Connector_PinHeader_2.54mm:PinHeader_1x02_P2.54mm_Vertical -> Connector_Dsub:DSUB-9_Female_Horizontal_P2.77x2.84mm_EdgePinOffset4.94mm_Housed_MountingHolesOffset7.48mm
- J4: value COM1: DCE -> COM2: DTE; footprint Connector_Dsub:DSUB-9_Female_Horizontal_P2.77x2.84mm_EdgePinOffset4.94mm_Housed_MountingHolesOffset7.48mm -> Connector_Dsub:DSUB-9_Male_Horizontal_P2.77x2.84mm_EdgePinOffset4.94mm_Housed_MountingHolesOffset7.48mm
- J5: value RTS/CTR DIR -> COM2 MAX BYPASS; footprint Connector_PinHeader_2.54mm:PinHeader_2x02_P2.54mm_Vertical -> Connector_PinHeader_2.54mm:PinHeader_2x03_P2.54mm_Vertical
- J6: value VCC DIS -> VCC BYPASS
- J7: value COM2: TTL -> COM2 TTL HANDSHAKE BYPASS; footprint Connector_PinHeader_2.54mm:PinHeader_1x06_P2.54mm_Horizontal -> Connector_PinHeader_2.54mm:PinHeader_2x05_P2.54mm_Vertical
- J8: value DATA DIR -> LATCH DELAY; footprint Connector_PinHeader_2.54mm:PinHeader_2x02_P2.54mm_Vertical -> Connector_PinHeader_2.54mm:PinHeader_1x03_P2.54mm_Vertical
- J9: value DTR|RTS/CTS -> COM2 BUS BYPASS; footprint Connector_PinHeader_2.54mm:PinHeader_1x03_P2.54mm_Vertical -> Connector_PinHeader_2.54mm:PinHeader_2x03_P2.54mm_Vertical
- RN1: footprint Resistor_THT:R_Array_SIP9 -> Resistor_THT:R_Array_SIP11
- RN2: footprint Resistor_THT:R_Array_SIP9 -> Resistor_THT:R_Array_SIP7
- RN3: value 3K3 -> 300; footprint Resistor_THT:R_Array_SIP5 -> Resistor_THT:R_Array_SIP9
- U1: value 74HC74 -> 74HCT74
- U11: value AS6C4008 -> Z84C4010; footprint Package_DIP:DIP-32_W15.24mm_Socket -> Package_DIP:DIP-40_W15.24mm_Socket
- U12: value Z84C3010 CTC -> MAX232; footprint Package_DIP:DIP-28_W15.24mm_Socket -> Package_DIP:DIP-16_W7.62mm_Socket
- U13: value MAX232 -> Z84C3010 CTC; footprint Package_DIP:DIP-16_W7.62mm_Socket -> Package_DIP:DIP-28_W15.24mm_Socket
- U14: value Z84C4010 -> MC14495; footprint Package_DIP:DIP-40_W15.24mm_Socket -> Package_DIP:DIP-16_W7.62mm_Socket
- U15: value Z84C20xx PIO -> MC14495; footprint Package_DIP:DIP-40_W15.24mm_Socket -> Package_DIP:DIP-16_W7.62mm_Socket
- U4: value ATF22V10C -> 74HCT573; footprint Package_DIP:DIP-24_W7.62mm_Socket -> Package_DIP:DIP-20_W7.62mm_Socket
- U7: value 74HCT573 -> Z84C0010; footprint Package_DIP:DIP-20_W7.62mm_Socket -> Package_DIP:DIP-40_W15.24mm_Socket
- U8: value Z84C0010 -> SST39SF010; footprint Package_DIP:DIP-40_W15.24mm_Socket -> 0_Library:DIP_Socket-32_W11.9_W12.7_W15.24_W17.78_W18.5_3M_232-1285-00-0602J
- U9: value SST39SF010 -> AS6C4008; footprint Socket:DIP_Socket-32_W11.9_W12.7_W15.24_W17.78_W18.5_3M_232-1285-00-0602J -> Package_DIP:DIP-32_W15.24mm_Socket
- X1: value 20 MHz -> 20MHz
- X2: value 3.6864 MHz -> 1.8432MHz
- moved X1 239.8 mm to (185.9, 64.1), turned to 90 degrees
- moved X2 234.9 mm to (186.0, 50.2), turned to 90 degrees
- moved C11 232.2 mm to (182.9, 103.5), turned to 90 degrees
- moved U1 231.4 mm to (186.1, 36.2), turned to 90 degrees
- moved C12 226.4 mm to (137.2, 59.1), turned to -90 degrees
- moved C1 221.2 mm to (182.2, 31.1), turned to -90 degrees
- moved C3 218.0 mm to (182.9, 45.1), turned to -90 degrees
- moved J3 216.8 mm to (239.4, 50.2)
- moved C2 209.1 mm to (182.8, 59.1), turned to -90 degrees
- moved U8 208.9 mm to (116.3, 33.7)
- moved C19 200.9 mm to (226.7, 40.0)
- moved C18 196.5 mm to (221.7, 40.0)
- moved C17 196.4 mm to (231.8, 40.0)
- moved C10 195.3 mm to (122.6, 81.9)
- moved U10 192.2 mm to (140.3, 43.8), turned to 90 degrees
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Connections:
- C13 pad 2: Net-(U13-VS+) -> GND
- C14 pad 1: Net-(U13-C1+) -> +5V
- C14 pad 2: Net-(U13-C1-) -> GND
- C15 pad 1: Net-(U13-C2+) -> +5V
- C15 pad 2: Net-(U13-C2-) -> GND
- C16 pad 1: Net-(U13-VS-) -> Net-(U12-C1+)
- C16 pad 2: GND -> Net-(U12-C1-)
- C17 pad 1: +5V -> Net-(U12-VS-)
- C18 pad 2: GND -> Net-(U12-VS+)
- C19 pad 1: +5V -> Net-(U12-C2+)
- C19 pad 2: GND -> Net-(U12-C2-)
- J1 pad 15: /IEO -> /SIO_IEI
- J1 pad 63: /~{BANK_CS} -> /~{BANK}
- J1 pad 72: /VCLK -> /CTCLK
- J1 pad 89: /TX2 -> /USR1
- J1 pad 90: /RX2 -> /USR2
- J1 pad 91: /USR1 -> /USR3
- J1 pad 92: /USR2 -> /USR4
- J1 pad 93: /USR3 -> /USR5
- J1 pad 94: /USR4 -> /USR6
- J1 pad 95: /USR5 -> /TX2
- J1 pad 97: /USR6 -> /RX2
- J11 pad 1: /CTC and SIO/TxB -> unconnected-(J11-Pad1)
- J11 pad 2: /TX -> /CTC and SIO/TX1
- J2 pad 1: /Glue Logic/~{MODE2_OE} -> /Glue Logic/~{MODE2OE}
- J4 pad 2: Net-(U13-T1out) -> /CTC and SIO/DB9Rx
- J4 pad 3: Net-(U13-R1in) -> /CTC and SIO/DB9Tx
- J4 pad 4: unconnected-(J4-Pad4) -> /CTC and SIO/DB9DTR
- J4 pad 7: Net-(U13-R2in) -> /CTC and SIO/DB9RTS
- J4 pad 8: Net-(U13-T2out) -> /CTC and SIO/DB9CTS
- J4 pad 9: unconnected-(J4-Pad9) -> Net-(J6-Pin_2)
- J5 pad 1: Net-(J5-Pin_1) -> /CTC and SIO/RxDB
- J5 pad 2: /CTC and SIO/~{CTSD} -> /CTC and SIO/TxDB
- J5 pad 3: /CTC and SIO/~{RTSD} -> /CTC and SIO/DB9Rx
- J5 pad 4: Net-(J5-Pin_4) -> /CTC and SIO/DB9Tx
- J7 pad 2: Net-(J5-Pin_4) -> unconnected-(J7-Pin_2-Pad2)
- J7 pad 3: Net-(J6-Pin_2) -> /CTC and SIO/~{CTSB}
- J7 pad 4: Net-(J7-Pin_4) -> /CTC and SIO/DB9CTS
- J7 pad 5: Net-(J7-Pin_5) -> /CTC and SIO/~{RTSB}
- J7 pad 6: Net-(J7-Pin_6) -> /CTC and SIO/DB9RTS
- J8 pad 1: /CTC and SIO/RxB -> /CLK
- J8 pad 2: Net-(J7-Pin_4) -> Net-(J8-Pin_2)
- J8 pad 3: Net-(J7-Pin_5) -> /~{CLK}
- J9 pad 1: Net-(J9-Pin_1) -> /CTC and SIO/RxB
- J9 pad 2: Net-(J7-Pin_6) -> /CTC and SIO/TxB
- J9 pad 3: Net-(J5-Pin_1) -> /CTC and SIO/RxDB
- RN2 pad 2: /~{IRQ}8 -> /~{IRQ}15
- RN2 pad 3: /~{IRQ}9 -> /~{IRQ}14
- RN2 pad 4: /~{IRQ}10 -> /~{IRQ}13
- RN2 pad 5: /~{IRQ}11 -> /~{IRQ}12
- RN2 pad 6: /~{IRQ}12 -> /~{IRQ}11
- RN2 pad 7: /~{IRQ}13 -> /~{IRQ}10
- RN3 pad 1: +5V -> GND
- RN3 pad 2: /~{WAIT} -> Net-(RN3-R1)
- RN3 pad 3: /~{BUSRQ} -> Net-(RN3-R2)
- RN3 pad 4: /~{INT} -> Net-(RN3-R3)
- RN3 pad 5: /~{NMI} -> Net-(RN3-R4)
- U1 pad 11: /CLK4 -> Net-(J8-Pin_2)
- U1 pad 12: Net-(U1B-D) -> /BANK_WR
- U1 pad 8: Net-(U1B-D) -> unconnected-(U1B-~{Q}-Pad8)
- U1 pad 9: /CLK2 -> /Blinkenlights/BANK_WR
- U10 pad 22: /~{RAM_CS1} -> /~{RAM_CS2}
- U11 pad 1: /BA18 -> /D1
- U11 pad 10: /A2 -> unconnected-(U11-~{W/RDYA}-Pad10)
- U11 pad 11: /A1 -> unconnected-(U11-~{SYNCA}-Pad11)
- U11 pad 12: /A0 -> /CTC and SIO/RxA
- U11 pad 13: /D0 -> /CTC and SIO/SIO_CLKA
- U11 pad 14: /D1 -> /CTC and SIO/SIO_CLKA
- U11 pad 15: /D2 -> /CTC and SIO/TxA
- U11 pad 16: GND -> unconnected-(U11-~{DTRA}-Pad16)
- U11 pad 17: /D3 -> unconnected-(U11-~{RTSA}-Pad17)
- U11 pad 18: /D4 -> GND
- U11 pad 19: /D5 -> GND
- U11 pad 2: /BA16 -> /D3
- U11 pad 20: /D6 -> /CLK
- U11 pad 21: /D7 -> /~{RESET}
- U11 pad 22: /~{RAM_CS2} -> GND
- U11 pad 23: /A10 -> /CTC and SIO/~{CTSB}
- U11 pad 24: /~{RD} -> /CTC and SIO/~{RTSB}
- U11 pad 25: /A11 -> /CTC and SIO/~{DTRB}
- U11 pad 26: /A9 -> /CTC and SIO/TxDB
- U11 pad 27: /A8 -> /CTC and SIO/SIO_CLKB
- U11 pad 28: /A13 -> /CTC and SIO/RxDB
- U11 pad 29: /~{WR} -> unconnected-(U11-~{SYNCB}-Pad29)
- U11 pad 3: /A14 -> /D5
- U11 pad 30: /BA17 -> unconnected-(U11-~{W/RDYB}-Pad30)
- U11 pad 31: /BA15 -> GND
- U11 pad 32: +5V -> /~{RD}
- U11 pad 4: /A12 -> /D7
- U11 pad 5: /A7 -> /~{IRQ}1
- U11 pad 6: /A6 -> /SIO_IEI
- U11 pad 7: /A5 -> /SIO_IEO
- U11 pad 8: /A4 -> /~{M1}
- U11 pad 9: /A3 -> +5V
- U12 pad 1: /D4 -> Net-(U12-C1+)
- U12 pad 10: /~{IORQ} -> /CTC and SIO/TxB
- U12 pad 11: unconnected-(U12-IEO-Pad11) -> /CTC and SIO/TxA
- U12 pad 12: /~{IRQ}0 -> /CTC and SIO/RxA
- U12 pad 13: /CTC and SIO/SIO_IEO -> /CTC and SIO/RX1
- U12 pad 14: /~{M1} -> /CTC and SIO/TX1
- U12 pad 15: /CLK -> GND
- U12 pad 16: /CTC_CS -> +5V
- U12 pad 2: /D5 -> Net-(U12-VS+)
- U12 pad 3: /D6 -> Net-(U12-C1-)
- U12 pad 4: /D7 -> Net-(U12-C2+)
- U12 pad 5: GND -> Net-(U12-C2-)
- U12 pad 6: /~{RD} -> Net-(U12-VS-)
- U12 pad 7: /VCLK -> /CTC and SIO/TxMAX
- U12 pad 8: /CTC and SIO/CTC_CLKA -> /CTC and SIO/RxMAX
- U12 pad 9: /CTC and SIO/CTC_CLKB -> /CTC and SIO/RxB
- U13 pad 1: Net-(U13-C1+) -> /D4
- U13 pad 10: /CTC and SIO/~{RTSA} -> /~{IORQ}
- U13 pad 11: /CTC and SIO/TxA -> unconnected-(U13-IEO-Pad11)
- U13 pad 12: /CTC and SIO/RxA -> /~{IRQ}0
- U13 pad 13: Net-(U13-R1in) -> /SIO_IEO
- U13 pad 14: Net-(U13-T1out) -> /~{M1}
- U13 pad 15: GND -> /CLK
- U13 pad 16: +5V -> /CTC_CS
- U13 pad 2: Net-(U13-VS+) -> /D5
- U13 pad 3: Net-(U13-C1-) -> /D6
- U13 pad 4: Net-(U13-C2+) -> /D7
- U13 pad 5: Net-(U13-C2-) -> GND
- U13 pad 6: Net-(U13-VS-) -> /~{RD}
- U13 pad 7: Net-(U13-T2out) -> /CTCLK
- U13 pad 8: Net-(U13-R2in) -> /CTC and SIO/CTC_CLKA
- U13 pad 9: /CTC and SIO/~{CTSA} -> /CTC and SIO/CTC_CLKB
- U14 pad 1: /D1 -> Net-(AFF2-e)
- U14 pad 10: unconnected-(U14-~{W/RDYA}-Pad10) -> /BA18
- U14 pad 12: /CTC and SIO/RxA -> Net-(AFF2-a)
- U14 pad 13: /CTC and SIO/SIO_CLKA -> Net-(AFF2-b)
- U14 pad 14: /CTC and SIO/SIO_CLKA -> Net-(AFF2-c)
- U14 pad 15: /CTC and SIO/TxA -> Net-(AFF2-d)
- U14 pad 16: unconnected-(U14-~{DTRA}-Pad16) -> +5V
- U14 pad 2: /D3 -> Net-(AFF2-f)
- U14 pad 3: /D5 -> Net-(AFF2-g)
- U14 pad 4: /D7 -> unconnected-(U14-H-Pad4)
- U14 pad 5: /~{IRQ}1 -> /BA15
- U14 pad 6: /PIO_IEO -> /BA16
- U14 pad 7: /CTC and SIO/SIO_IEO -> /Blinkenlights/BANK_WR
- U14 pad 8: /~{M1} -> GND
- U14 pad 9: +5V -> /BA17
- U15 pad 1: /D2 -> Net-(AFF1-e)
- U15 pad 10: /PIO/ROW5 -> /BA22
- U15 pad 11: GND -> unconnected-(U15-I-Pad11)
- U15 pad 12: /PIO/ROW4 -> Net-(AFF1-a)
- U15 pad 13: /PIO/ROW3 -> Net-(AFF1-b)
- U15 pad 14: /PIO/ROW2 -> Net-(AFF1-c)
- U15 pad 15: /PIO/ROW1 -> Net-(AFF1-d)
- U15 pad 16: unconnected-(U15-~{ASTB}-Pad16) -> +5V
- U15 pad 2: /D7 -> Net-(AFF1-f)
- U15 pad 3: /D6 -> Net-(AFF1-g)
- U15 pad 4: /PIO_CS -> unconnected-(U15-H-Pad4)
- U15 pad 5: /A1 -> /BA19
- U15 pad 6: /A0 -> /BA20
- U15 pad 7: /PIO/ROW8 -> /Blinkenlights/BANK_WR
- U15 pad 8: /PIO/ROW7 -> GND
- U15 pad 9: /PIO/ROW6 -> /BA21
- U2 pad 1: /~{MREQ} -> /~{RESET}
- U2 pad 10: /A6 -> /A5
- U2 pad 11: /A7 -> /A6
- U2 pad 13: /~{RESET} -> /A7
- U2 pad 17: /~{BANK_CS} -> /~{BANK}
- U2 pad 18: unconnected-(U2-I/O-Pad18) -> /SIO_CS
- U2 pad 19: /Glue Logic/~{MODE2_OE} -> /CTC_CS
- U2 pad 2: /~{IORQ} -> /~{MREQ}
- U2 pad 20: /Glue Logic/~{ROM_DIS} -> /Glue Logic/~{BANK_RD}
- U2 pad 21: /Glue Logic/~{INT_RD} -> /BANK_WR
- U2 pad 22: /Glue Logic/~{BANK_RD} -> /Glue Logic/~{INT_RD}
- U2 pad 23: /Glue Logic/BANK_SEL -> /Glue Logic/~{MODE2OE}
- U2 pad 3: /~{M1} -> /~{IORQ}
- U2 pad 4: /~{WR} -> /~{M1}
- U2 pad 5: /~{RD} -> /~{WR}
- U2 pad 6: /A2 -> /~{RD}
- U2 pad 7: /A3 -> /A2
- U2 pad 8: /A4 -> /A3
- U2 pad 9: /A5 -> /A4
- U3 pad 1: /~{IORQ} -> /~{IRQ}0
- U3 pad 10: /A7 -> /~{IRQ}9
- U3 pad 11: GND -> /~{IRQ}10
- U3 pad 13: GND -> /~{IRQ}11
- U3 pad 14: unconnected-(U3-I/O-Pad14) -> /~{IRQ}12
- U3 pad 15: unconnected-(U3-I/O-Pad15) -> /~{IRQ}13
- U3 pad 16: unconnected-(U3-I/O-Pad16) -> /~{IRQ}14
- U3 pad 17: unconnected-(U3-I/O-Pad17) -> /~{IRQ}15
- U3 pad 19: unconnected-(U3-I/O-Pad19) -> Net-(D1-K)
- U3 pad 2: /~{M1} -> /~{IRQ}1
- U3 pad 20: unconnected-(U3-I/O-Pad20) -> Net-(U4-D4)
- U3 pad 21: /PIO_CS -> Net-(U4-D3)
- U3 pad 22: /SIO_CS -> Net-(U4-D2)
- U3 pad 23: /CTC_CS -> Net-(U4-D1)
- U3 pad 3: /~{WR} -> /~{IRQ}2
- U3 pad 4: /~{RD} -> /~{IRQ}3
- U3 pad 5: /A2 -> /~{IRQ}4
- U3 pad 6: /A3 -> /~{IRQ}5
- U3 pad 7: /A4 -> /~{IRQ}6
- U3 pad 8: /A5 -> /~{IRQ}7
- U3 pad 9: /A6 -> /~{IRQ}8
- U4 pad 1: /Glue Logic/BANK_SEL -> Net-(J2-Pin_2)
- U4 pad 10: /A15 -> GND
- U4 pad 11: /~{BANK_CS} -> /~{M1}
- U4 pad 12: GND -> /D7
- U4 pad 13: /~{RESET} -> /D6
- U4 pad 14: /~{RAM_CS2} -> /D5
- U4 pad 15: /~{RAM_CS1} -> /D4
- U4 pad 16: /BA22 -> /D3
- U4 pad 17: /BA21 -> /D2
- U4 pad 18: /BA20 -> /D1
- U4 pad 19: /BA19 -> /D0
- U4 pad 2: /D0 -> GND
- U4 pad 20: /BA18 -> +5V
- U4 pad 3: /D1 -> Net-(U4-D1)
- U4 pad 4: /D2 -> Net-(U4-D2)
- U4 pad 5: /D3 -> Net-(U4-D3)
- U4 pad 6: /D4 -> Net-(U4-D4)
- U4 pad 7: /D5 -> GND
- U4 pad 8: /D6 -> GND
- U4 pad 9: /D7 -> GND
- U5 pad 1: /~{IRQ}0 -> /BANK_WR
- U5 pad 10: /~{IRQ}9 -> /A15
- U5 pad 11: /~{IRQ}10 -> /~{BANK}
- U5 pad 13: /~{IRQ}11 -> /~{RESET}
- U5 pad 14: /~{IRQ}12 -> /~{RAM_CS2}
- U5 pad 15: /~{IRQ}13 -> /~{RAM_CS1}
- U5 pad 16: /~{IRQ}14 -> /BA22
- U5 pad 17: /~{IRQ}15 -> /BA21
- U5 pad 18: unconnected-(U5-I/O-Pad18) -> /BA20
- U5 pad 19: /~{INT} -> /BA19
- U5 pad 2: /~{IRQ}1 -> /D0
- U5 pad 20: Net-(U7-D4) -> /BA18
- U5 pad 21: Net-(U7-D3) -> /BA17
- U5 pad 22: Net-(U7-D2) -> /BA16
- U5 pad 23: Net-(U7-D1) -> /BA15
- U5 pad 3: /~{IRQ}2 -> /D1
- U5 pad 4: /~{IRQ}3 -> /D2
- U5 pad 5: /~{IRQ}4 -> /D3
- U5 pad 6: /~{IRQ}5 -> /D4
- U5 pad 7: /~{IRQ}6 -> /D5
- U5 pad 8: /~{IRQ}7 -> /D6
- U5 pad 9: /~{IRQ}8 -> /D7
- U7 pad 1: Net-(J2-Pin_2) -> /A11
- U7 pad 10: GND -> /D6
- U7 pad 11: /~{M1} -> +5V
- U7 pad 12: /D7 -> /D2
- U7 pad 13: /D6 -> /D7
- U7 pad 14: /D5 -> /D0
- U7 pad 15: /D4 -> /D1
- U7 pad 16: /D3 -> /~{INT}
- U7 pad 17: /D2 -> /~{NMI}
- U7 pad 18: /D1 -> /~{HALT}
- U7 pad 19: /D0 -> /~{MREQ}
- U7 pad 2: GND -> /A12
- U7 pad 20: +5V -> /~{IORQ}
- U7 pad 3: Net-(U7-D1) -> /A13
- U7 pad 4: Net-(U7-D2) -> /A14
- U7 pad 5: Net-(U7-D3) -> /A15
- U7 pad 6: Net-(U7-D4) -> /CLK
- U7 pad 7: GND -> /D4
- U7 pad 8: GND -> /D3
- U7 pad 9: GND -> /D5
- U8 pad 1: /A11 -> unconnected-(U8-NC-Pad1)
- U8 pad 10: /D6 -> /A2
- U8 pad 11: +5V -> /A1
- U8 pad 12: /D2 -> /A0
- U8 pad 13: /D7 -> /D0
- U8 pad 14: /D0 -> /D1
- U8 pad 15: /D1 -> /D2
- U8 pad 16: /~{INT} -> GND
- U8 pad 17: /~{NMI} -> /D3
- U8 pad 18: /~{HALT} -> /D4
- U8 pad 19: /~{MREQ} -> /D5
- U8 pad 2: /A12 -> GND
- U8 pad 20: /~{IORQ} -> /D6
- U8 pad 21: /~{RD} -> /D7
- U8 pad 22: /~{WR} -> /~{ROM_CS}
- U8 pad 23: /~{BUSAK} -> /A10
- U8 pad 24: /~{WAIT} -> /~{RD}
- U8 pad 25: /~{BUSRQ} -> /A11
- U8 pad 26: /~{RESET} -> /A9
- U8 pad 27: /~{M1} -> /A8
- U8 pad 28: unconnected-(U8-~{RFSH}-Pad28) -> /A13
- U8 pad 29: GND -> /A14
- U8 pad 3: /A13 -> /A15
- U8 pad 30: /A0 -> unconnected-(U8-NC-Pad30)
- U8 pad 31: /A1 -> /~{WR}
- U8 pad 32: /A2 -> +5V
- U8 pad 4: /A14 -> /A12
- U8 pad 5: /A15 -> /A7
- U8 pad 6: /CLK -> /A6
- U8 pad 7: /D4 -> /A5
- U8 pad 8: /D3 -> /A4
- U8 pad 9: /D5 -> /A3
- U9 pad 1: unconnected-(U9-NC-Pad1) -> /BA18
- U9 pad 2: GND -> /BA16
- U9 pad 22: /~{ROM_CS} -> /~{RAM_CS1}
- U9 pad 29: /A14 -> /~{WR}
- U9 pad 3: /A15 -> /A14
- U9 pad 30: unconnected-(U9-NC-Pad30) -> /BA17
- U9 pad 31: /~{WR} -> /BA15
- X2 pad 5: /CLK4 -> /CLK2
Other:
- board size 152.3 x 106.7 mm -> 174.4 x 99.1 mm
