File: 2 - CPU and memory card with the essentials (rev 2)/Blinkenlights.kicad_sch (KiCad schematic)
At the start: 10 parts, among them U14 MC14495, U15 MC14495, U16 74HCT563

Commit message: Trying to hash out the flaws
Parts:
- removed AFF1: HI BANK #, Display_7Segment:7SegmentLED_LTS6760_LTS6780, symbol Display_Character:LTS-6980HR
- removed AFF2: LO BANK #, Display_7Segment:7SegmentLED_LTS6760_LTS6780, symbol Display_Character:LTS-6980HR
- removed BAR1: STATUS, 0_Library:BAR_GRAPH_8, symbol 0_Library:BAR_GRAPH_8
- removed C14, C15: 0.1µF, Capacitor_THT:C_Disc_D3.0mm_W1.6mm_P2.50mm, symbol Device:C
- removed RN3: 300, Resistor_THT:R_Array_SIP9, symbol Device:R_Network08_US
- removed U14, U15: MC14495, Package_DIP:DIP-16_W7.62mm_Socket, symbol 0_Library:MC14495
- removed U16: 74HCT563, Package_DIP:DIP-20_W7.62mm_Socket, symbol 0_Library:74HC563
Connections:
- no-connect marks 6 -> 0
Other:
- note added: "Bypass Capacitor"
- note removed: "BANK DISPLAY"
- note removed: "BLINKENLIGHTS"
- note removed: "Bypass Capacitors"
