File: 2 - CPU and core components (Rev 2)/Blinkenlights.kicad_sch (KiCad schematic)
At the start: 3 parts, among them U17 74HCT240

Commit message: Added Interrupt Enable daisy chain jumpers between the ISA slots
Other:
- company: (none) -> Frédéric Segard
Changed lines of the file:
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@@
 (kicad_sch (version 20230121) (generator eeschema)
-  (paper "A4")
+  (paper "USLetter")
+  (title_block
+    (date "2023-08-29")
+    (rev "2")
+    (company "Frédéric Segard")
+    (comment 1 "@microhobbyist")
+    (comment 4 "Thank you to John Winans for his inspiration, as well as Grant Searle and Sergey Kiselev")
+  )
   (junction (at 151.13 105.41) (diameter 0) (color 0 0 0 0)
   )

Commit message: Finished component placement, currently routing.
Parts:
- added C?: 1µF, Capacitor_THT:C_Disc_D3.4mm_W2.1mm_P2.50mm, symbol Device:C
Connections:
- net +5V: now also C?.1
- net GND: now also C?.2
Other:
- note added: "Bypass Capacitor"
- moved on the sheet: BAR1, RN5, U17
