File: 2 - CPU and core components (Rev 2)/CTC.kicad_sch (KiCad schematic)
At the start: 2 parts

Commit message: Finished component placement, currently routing.
Other:
- note added: "Bypass Capacitor"
- note removed: "Bypass Capacitors"
Changed lines of the file:
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@@
     (effects (font (size 2 2) (thickness 0.508) bold italic) (justify left bottom))
   )
-  (text "Bypass Capacitors" (at 19.05 184.15 0)
+  (text "Bypass Capacitor" (at 19.05 184.15 0)
     (effects (font (size 1.27 1.27)) (justify left bottom))
   )
