File: 2 - CPU and core components (Rev 2.1)/2 - CPU and core components (Rev 2.1).kicad_sch (KiCad schematic)
At the start: 12 parts

Commit message: Trying to work out the PLD logic
Parts:
- removed C?: 1µF, Capacitor_THT:C_Disc_D3.4mm_W2.1mm_P2.50mm, symbol Device:C
- removed RN4: 3K3, Resistor_THT:R_Array_SIP9, symbol Device:R_Network08_US
- removed U?: 74LS245, Package_DIP:DIP-20_W7.62mm_Socket, symbol 74xx:74LS245
- added RN?: 3K3, Resistor_THT:R_Array_SIP11, symbol Device:R_Network10_US
Connections:
- net USR8 is gone; now on net ~{RAM_OE}: J?.97 (D17)
- net +5V: now also RN?.1 (common)
- net A0: now also U?.18 (B0); no longer U?.2 (A0)
- net A1: now also U?.17 (B1); no longer U?.3 (A1)
- net A10: now also U?.16 (B2); no longer U?.4 (A2)
- net A11: now also U?.15 (B3); no longer U?.5 (A3)
- net A12: now also U?.14 (B4); no longer U?.6 (A4)
- net A13: now also U?.13 (B5); no longer U?.7 (A5)
- net A14: now also U?.12 (B6); no longer U?.8 (A6)
- net A15: now also U?.11 (B7); no longer U?.9 (A7)
- net A2: now also U?.16 (B2); no longer U?.4 (A2)
- net A3: now also U?.15 (B3); no longer U?.5 (A3)
- net A4: now also U?.14 (B4); no longer U?.6 (A4)
- net A5: now also U?.13 (B5); no longer U?.7 (A5)
- net A6: now also U?.12 (B6); no longer U?.8 (A6)
- net A7: now also U?.11 (B7); no longer U?.9 (A7)
- net A8: now also U?.18 (B0); no longer U?.2 (A0)
- net A9: now also U?.17 (B1); no longer U?.3 (A1)
- net BUS_IEI: now also RN?.11 (R10)
- net BufA0: now also U?.2 (A0); no longer U?.18 (B0)
- net BufA1: now also U?.3 (A1); no longer U?.17 (B1)
- net BufA10: now also U?.4 (A2); no longer U?.16 (B2)
- net BufA11: now also U?.5 (A3); no longer U?.15 (B3)
- net BufA12: now also U?.6 (A4); no longer U?.14 (B4)
- net BufA13: now also U?.7 (A5); no longer U?.13 (B5)
- net BufA14: now also U?.8 (A6); no longer U?.12 (B6)
- net BufA15: now also U?.9 (A7); no longer U?.11 (B7)
- net BufA2: now also U?.4 (A2); no longer U?.16 (B2)
- net BufA3: now also U?.5 (A3); no longer U?.15 (B3)
- net BufA4: now also U?.6 (A4); no longer U?.14 (B4)
- net BufA5: now also U?.7 (A5); no longer U?.13 (B5)
- net BufA6: now also U?.8 (A6); no longer U?.12 (B6)
- net BufA7: now also U?.9 (A7); no longer U?.11 (B7)
- net BufA8: now also U?.2 (A0); no longer U?.18 (B0)
- net BufA9: now also U?.3 (A1); no longer U?.17 (B1)
- net GND: no longer U?.1 (OEa), U?.13 (I1b), U?.15 (I2b), U?.17 (I3b)
- net ~{BUSAK}: now also U?.15 (I2b); no longer U?.1 (A->B), U?.1 (A->B), U?.6 (I2a)
- net ~{BUSRQ}: now also J?.47 (B16), RN?.6 (R5); no longer U?.12 (O3a)
- net ~{BufBUSAK}: now also U?.5 (O2b); no longer U?.14 (O2a)
- net ~{BufHALT}: now also U?.7 (O1b); no longer U?.16 (O1a)
- net ~{BufIORQ}: now also U?.16 (O1a), RN?.3 (R2)
- net ~{BufM1}: now also U?.9 (O0b); no longer U?.18 (O0a)
- net ~{BufMREQ}: now also U?.18 (O0a), RN?.2 (R1)
- net ~{BufRD}: now also J?.44 (B13), U?.14 (O2a), RN?.4 (R3); no longer J?.45 (B14)
- net ~{BufWAIT}: now also U?.17 (I3b); no longer U?.11 (I0b)
- net ~{BufWR}: now also J?.45 (B14), U?.12 (O3a), RN?.5 (R4); no longer J?.44 (B13)
- net ~{HALT}: now also U?.13 (I1b); no longer U?.4 (I1a)
- net ~{IORQ}: now also U?.4 (I1a)
- net ~{M1}: now also U?.11 (I0b); no longer U?.2 (I0a)
- net ~{MREQ}: now also U?.2 (I0a)
- net ~{NMI}: now also RN?.9 (R8)
- net ~{RAM_OE}: no longer J?.64 (C2)
- net ~{RD}: now also U?.6 (I2a)
- net ~{WAIT}: now also U?.3 (O3b), RN?.7 (R6); no longer U?.9 (O0b)
- net ~{WR}: now also U?.8 (I3a)
- net DIR renamed BufDIR
- removed net ~{BufBUSRQ}: J?.47 (B16), U?.8 (I3a)
- new net !BUSAK: U?.1 (A->B), U?.1 (A->B), U?.1 (OEa)
- new net BA22: J?.64 (C2)
- new net CTC_IEI: RN?.10 (R9)
- new net ~{INT}: RN?.8 (R7)
- no-connect marks 29 -> 25
Other:
- moved on the sheet: U?
