File: 2 - CPU and core components (Rev 2.1)/CPUandMemory.kicad_sch (KiCad schematic)
At the start: 11 parts, among them U22 74LS30

Commit message: Trying to work out the PLD logic
Parts:
- removed RN?: 3K3, Resistor_THT:R_Array_SIP9, symbol Device:R_Network08_US
Connections:
- net ~{RD}: no longer U?.24 (~{OE})
- net ~{WR}: no longer U?.29 (~{WE}), U?.31 (~{PGM})
- new net ~{BufRD}: U?.24 (~{OE})
- new net ~{BufWR}: U?.29 (~{WE}), U?.31 (~{PGM})
