File: 2 - CPU and core components (Rev 2.1)/GlueLogic.kicad_sch (KiCad schematic)
At the start: 32 parts, among them J2 INT MODE, U10 ATF22V10C, U11 74HCT373, U12 74LS273, U14 74HCT373, U6 74HCT132, U7 74HCT74, U8 74HCT32, U9 ATF22V10C

Commit message: Trying to work out the PLD logic
Parts:
- removed C?: 1µF, Capacitor_THT:C_Disc_D3.0mm_W2.0mm_P2.50mm, symbol Device:C
- removed U6: 74HCT132, Package_DIP:DIP-14_W7.62mm_Socket, symbol 74xx:74LS132
- removed U8, U? (x3): 74HCT32, Package_DIP:DIP-14_W7.62mm_Socket, symbol 74xx:74LS32
- added U2: ATF16V8B, Package_DIP:DIP-20_W7.62mm_Socket, symbol 0_Library:ATF16V8B
Connections:
- net DIR is gone; now on net ~{RAM_CS}: U10.18 (I/O)
- net ~{IORQ} is gone; now on net ~{M1}: U10.3 (I)
- net ~{RD} is gone; now on net A15: U10.6 (I)
- net +5V: now also U2.20 (VCC)
- net A15: no longer U10.13 (I)
- net BA19: now also U10.13 (I); no longer U10.14 (I/O)
- net BA20: now also U10.14 (I/O); no longer U10.15 (I/O)
- net BA21: now also U10.15 (I/O); no longer U10.16 (I/O)
- net D7: now also U12.18 (D7)
- net GND: now also U2.10 (GND); no longer U12.18 (D7)
- net ~{IRQ}0: now also U2.5 (I)
- net ~{IRQ}1: now also U2.6 (I)
- net ~{M1}: now also U2.3 (I); no longer U10.4 (I/PD)
- net ~{MODE1}: now also U2.9 (I)
- net ~{RAM_CS}: no longer U10.17 (I/O)
- net ~{RAM_OE}: now also U2.17 (I/O)
- net ~{RESET}: now also U2.8 (I)
- net ~{ROM_CS}: now also U2.18 (I/O)
- net BA22: now reaches U12.19 (Q7)
- net BA22: now also U10.16 (I/O)
- net ~{BUSAK} renamed ~{BufMREQ}
- net ~{BufMREQ}: now also U2.1 (I/CLK)
- net ~{MODE0/2} renamed ~{MODE2}
- net ~{MODE2}: now also U2.13 (I/O)
- net ~{MREQ} renamed ~{BufIORQ}
- net ~{BufIORQ}: now also U2.2 (I)
- net ~{WR} renamed ~{BufRD}
- net ~{BufRD}: now also U2.4 (I)
- new net !BUSAK: U2.12 (I/O)
- new net BufDIR: U2.19 (I/O)
- new net ~{BufBUSAK}: U2.7 (I)
- new net ~{BufWR}: U10.4 (I/PD)
- new net ~{IOSEL}: U10.17 (I/O), U2.11 (I/~{OE})
- no-connect marks 5 -> 4
Other:
- note added: "(~{ROMDIS})"
- note added: "00-1Fh"
- note added: "10-17h"
- note added: "18-1Fh (~{ROMDIS})"
- note added: "Reserved"
- note added: "SHADOW AND BUFFER DIRECTION LOGIC"
- note removed: "30-37h"
- note removed: "38-3Fh (~{ROMDIS})"
- note removed: "SHADOW LOGIC"
- note removed: "~{ROM_DIS}"
- moved on the sheet: J2, U10, U14, U7A, U7B, X?
