File: 2 - CPU and core components (Rev 2.1)/SIO.kicad_sch (KiCad schematic)
At the start: 25 parts

Commit message: Trying to work out the PLD logic
Parts:
- added R? (x2): 3K3, Resistor_THT:R_Axial_DIN0207_L6.3mm_D2.5mm_P10.16mm_Horizontal, symbol Device:R_US
- R? (x2): value 150 -> 120
Connections:
- net +5V: now also R?.2, R?.2
- net R_FTRA: no longer names the net of D?.2 (A)
- net R_FTRA: now also R?.1
- net R_FTRB: no longer names the net of D?.2 (A)
- net R_FTRB: now also R?.1
- net ~{IORQ} renamed ~{BufIORQ}
- net ~{RD} renamed ~{BufRD}
